File: Mini drone/Mini drone.kicad_sch (KiCad schematic)
At the start: 37 parts, among them J1 USB_C_Receptacle_USB2.0_16P, J2 JST_2mm_LiPo, J3 Conn_01x06_Socket, J4 Conn_01x06_Socket, Q1 AO3401A, SW1 SW_DPDT_x2, U1 ESP32-WROOM-32, U2 MIC5219-3.3YM5, U3 TP4056-42-ESOP8

Commit message: 21-06-2025
Other:
- note added: "3.3v Regulator"
- note added: "External connector"
- note added: "MCU"
- note added: "Switch"
- note added: "TP4056"
Changed lines of the file:
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@@
 		(rev "1")
 	)
-	(text_box "3.3v Regulator\n"
+	(text "TP4056"
 		(exclude_from_sim no)
-		(at 20.0025 12.7 0)
-		(size 140.0175 75.565)
-		(margins 0.9525 0.9525 0.9525 0.9525)
-		(stroke
-			(width 0)
-			(type solid)
-		)
-		(fill
-			(type none)
-		)
-		(effects
-			(font
-				(size 1.27 1.27)
-			)
-			(justify left top)
-		)
-	)
-	(text_box "MCU\n"
+		(at 180.34 20.32 0)
+		(effects
+			(font
+				(size 1.27 1.27)
+			)
+		)
+	)
+	(text "External connector\n"
 		(exclude_from_sim no)
-		(at 20.32 94.9325 0)
-		(size 114.3 86.995)
-		(margins 0.9525 0.9525 0.9525 0.9525)
-		(stroke
-			(width 0)
-			(type solid)
-		)
-		(fill
-			(type none)
-		)
-		(effects
-			(font
-				(size 1.27 1.27)
-			)
-			(justify left top)
-		)
-	)
-	(text_box "External connector\n"
+		(at 157.629 136.4936 0)
+		(effects
+			(font
+				(size 1.27 1.27)
+			)
+		)
+	)
+	(text "MCU"
 		(exclude_from_sim no)
-		(at 145.415 135.5725 0)
-		(size 71.755 26.3525)
-		(margins 0.9525 0.9525 0.9525 0.9525)
-		(stroke
-			(width 0)
-			(type solid)
-		)
-		(fill
-			(type none)
-		)
-		(effects
-			(font
-				(size 1.27 1.27)
-			)
-			(justify left top)
-		)
-	)
-	(text_box "TP4056"
+		(at 25.4 95.25 0)
+		(effects
+			(font
+				(size 1.27 1.27)
+			)
+		)
+	)
+	(text "Switch"
 		(exclude_from_sim no)
-		(at 171.7675 18.0975 0)
-		(size 103.8225 45.4025)
-		(margins 0.9525 0.9525 0.9525 0.9525)
-		(stroke
-			(width 0)
-			(type solid)
-		)
-		(fill
-			(type none)
-		)
-		(effects
-			(font
-				(size 1.27 1.27)
-			)
-			(justify left top)
-		)
-	)
-	(text_box "Switch"
+		(at 163.83 96.52 0)
+		(effects
+			(font
+				(size 1.27 1.27)
+			)
+		)
+	)
+	(text "3.3v Regulator\n"
 		(exclude_from_sim no)
-		(at 158.75 93.6625 0)
-		(size 42.545 39.0525)
-		(margins 0.9525 0.9525 0.9525 0.9525)
-		(stroke
-			(width 0)
-			(type solid)
-		)
-		(fill
-			(type none)
-		)
-		(effects
-			(font
-				(size 1.27 1.27)
-			)
-			(justify left top)
+		(at 29.21 15.24 0)
+		(effects
+			(font
+				(size 1.27 1.27)
+			)
 		)
 	)
@@
 			)
 		)
+	)
+	(rule_area
+		(polyline
+			(pts
+				(xy 160.02 93.98) (xy 198.12 93.98) (xy 198.12 132.08) (xy 160.02 132.08)
+			)
+			(stroke
+				(width 0)
+				(type dash)
+			)
+			(fill
+				(type none)
+			)
+		)
+	)
+	(rule_area
+		(polyline
+			(pts
+				(xy 147.32 134.62) (xy 217.17 134.62) (xy 217.17 160.02) (xy 147.32 160.02)
+			)
+			(stroke
+				(width 0)
+				(type dash)
+			)
+			(fill
+				(type none)
+			)
+		)
+	)
+	(rule_area
+		(polyline
+			(pts
+				(xy 21.59 92.71) (xy 21.59 182.88) (xy 134.62 182.88) (xy 134.62 92.71)
+			)
+			(stroke
+				(width 0)
+				(type dash)
+			)
+			(fill
+				(type none)
+			)
+		)
+	)
+	(rule_area
+		(polyline
+			(pts
+				(xy 20.32 12.7) (xy 160.02 12.7) (xy 161.29 12.7) (xy 161.29 88.9) (xy 20.32 88.9)
+			)
+			(stroke
+				(width 0)
+				(type dash)
+			)
+			(fill
+				(type none)
+			)
+		)
+	)
+	(rule_area
+		(polyline
+			(pts
+				(xy 175.3364 18.3968) (xy 273.1264 18.3968) (xy 273.1264 62.8468) (xy 175.3364 62.8468)
+			)
+			(stroke
+				(width 0)
+				(type dash)
+			)
+			(fill
+				(type none)
+			)
+		)
