File: Mini drone/debugUSB.kicad_sch (KiCad schematic)
At the start: 17 parts, among them U4 CP2102N-Axx-xQFN28, U5 DDC114TU-7-F, U6 MPU-6050

Commit message: 21-06-2025
Other:
- note added: "CP2102 USB debug"
- note added: "MPU 6050"
Changed lines of the file:
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@@
 		(rev "1")
 	)
-	(text_box "CP2102 USB debug"
+	(text "CP2102 USB debug"
 		(exclude_from_sim no)
-		(at 37.465 32.385 0)
-		(size 99.06 123.5075)
-		(margins 0.9525 0.9525 0.9525 0.9525)
-		(stroke
-			(width 0)
-			(type solid)
-		)
-		(fill
-			(type none)
-		)
-		(effects
-			(font
-				(size 1.27 1.27)
-			)
-			(justify left top)
-		)
-	)
-	(text_box "MPU 6050"
+		(at 49.53 39.37 0)
+		(effects
+			(font
+				(size 1.27 1.27)
+			)
+		)
+	)
+	(text "MPU 6050"
 		(exclude_from_sim no)
-		(at 148.9075 56.1975 0)
-		(size 120.3325 70.8025)
-		(margins 0.9525 0.9525 0.9525 0.9525)
-		(stroke
-			(width 0)
-			(type solid)
-		)
-		(fill
-			(type none)
-		)
-		(effects
-			(font
-				(size 1.27 1.27)
-			)
-			(justify left top)
+		(at 154.94 59.69 0)
+		(effects
+			(font
+				(size 1.27 1.27)
+			)
 		)
 	)
@@
 		)
 	)
+	(rule_area
+		(polyline
+			(pts
+				(xy 38.1 36.83) (xy 135.89 36.83) (xy 135.89 151.13) (xy 135.89 152.4) (xy 38.1 152.4)
+			)
+			(stroke
+				(width 0)
+				(type dash)
+			)
+			(fill
+				(type none)
+			)
+		)
+	)
+	(rule_area
+		(polyline
+			(pts
+				(xy 148.59 57.15) (xy 269.24 57.15) (xy 269.24 120.65) (xy 148.59 120.65) (xy 148.59 116.84)
+			)
+			(stroke
+				(width 0)
+				(type dash)
+			)
+			(fill
+				(type none)
+			)
+		)
+	)
