File: Mini drone/motor_driver.kicad_sch (KiCad schematic)
At the start: 18 parts, among them J5 Conn_01x02_Socket, J6 Conn_01x02_Socket, J7 Conn_01x02_Socket, J8 Conn_01x02_Socket, U7 DRV8833PWP, U8 DRV8833PWP, U9 PCF8574ATS

Commit message: 21-06-2025
Other:
- note added: "DRV8833 motor driver"
- note added: "PCF8574 8bit expander"
Changed lines of the file:
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@@
 		(rev "1")
 	)
-	(text_box "DRV8833 motor driver\n"
+	(text "PCF8574 8bit expander"
 		(exclude_from_sim no)
-		(at 31.75 22.86 0)
-		(size 236.5375 63.5)
-		(margins 0.9525 0.9525 0.9525 0.9525)
-		(stroke
-			(width 0)
-			(type solid)
-		)
-		(fill
-			(type none)
-		)
-		(effects
-			(font
-				(size 1.27 1.27)
-			)
-			(justify left top)
-		)
-	)
-	(text_box "PCF8574 8bit expander"
+		(at 142.24 93.98 0)
+		(effects
+			(font
+				(size 1.27 1.27)
+			)
+		)
+	)
+	(text "DRV8833 motor driver\n"
 		(exclude_from_sim no)
-		(at 98.1075 89.2175 0)
-		(size 66.04 63.5)
-		(margins 0.9525 0.9525 0.9525 0.9525)
-		(stroke
-			(width 0)
-			(type solid)
-		)
-		(fill
-			(type none)
-		)
-		(effects
-			(font
-				(size 1.27 1.27)
-			)
-			(justify left top)
+		(at 45.72 21.59 0)
+		(effects
+			(font
+				(size 1.27 1.27)
+			)
 		)
 	)
@@
 	(wire
 		(pts
-			(xy 116.84 95.25) (xy 116.84 115.57)
+			(xy 116.84 97.79) (xy 116.84 115.57)
 		)
 		(stroke
@@
 	(wire
 		(pts
-			(xy 119.38 100.33) (xy 119.38 107.95)
+			(xy 119.38 101.6) (xy 119.38 107.95)
 		)
 		(stroke
@@
 	(hierarchical_label "SDA"
 		(shape bidirectional)
-		(at 116.84 95.25 90)
+		(at 116.84 97.79 90)
 		(effects
 			(font
@@
 	(hierarchical_label "SCL"
 		(shape bidirectional)
-		(at 119.38 100.33 90)
+		(at 119.38 101.6 90)
 		(effects
 			(font
@@
 		)
 	)
+	(rule_area
+		(polyline
+			(pts
+				(xy 33.02 19.05) (xy 260.35 19.05) (xy 261.9375 19.05) (xy 261.62 85.09) (xy 33.02 85.09)
+			)
+			(stroke
+				(width 0)
+				(type dash)
+			)
+			(fill
+				(type none)
+			)
+		)
+	)
+	(rule_area
+		(polyline
+			(pts
+				(xy 102.87 91.44) (xy 153.67 91.44) (xy 153.67 152.4) (xy 152.4 152.4) (xy 102.87 152.4)
+			)
+			(stroke
+				(width 0)
+				(type dash)
+			)
+			(fill
+				(type none)
+			)
+		)
+	)
