File: Mini drone/Mini drone.kicad_pcb (KiCad board)
At the start: 2 copper layers, 102.4 x 102.4 mm, 72 parts, among them J1 USB_C_Receptacle_USB2.0_16P, J2 JST_2mm_LiPo, J3 Conn_01x06_Socket, J4 Conn_01x06_Socket, J5 Conn_01x02_Socket, J6 Conn_01x02_Socket, J7 Conn_01x02_Socket, J8 Conn_01x02_Socket, Q1 AO3401A, SW1 SW_DPDT_x2, U1 ESP32-WROOM-32, U2 MIC5219-3.3YM5, U3 TP4056-42-ESOP8, U4 CP2102N-Axx-xQFN28, U5 DDC114TU-7-F, U6 MPU-6050, U7 DRV8833PWP, U8 DRV8833PWP, U9 PCF8574ATS

Commit message: 07-08-2025
Parts:
- moved U6 7.63 mm to (226.1, 104.7)
- moved C12 5.74 mm to (233.7, 106.7)
- moved C13 5.62 mm to (233.6, 104.5)
- moved C11 5.56 mm to (233.5, 102.3)
- moved C14 3.32 mm to (207.5, 101.6), turned to 180 degrees
- moved R24 3.22 mm to (211.4, 101.7)
- moved R25 3.22 mm to (211.4, 103.9)
- moved R26 3.22 mm to (211.4, 106.2)
- moved C15 2.85 mm to (207.5, 103.8)
- moved C16 2.85 mm to (207.5, 106.3)
- moved U9 2.54 mm to (218.4, 104.5)
- moved R1 1.12 mm to (238.9, 100.6)
- moved R21 1.12 mm to (238.9, 102.5)
- moved R19 1.12 mm to (238.9, 106.3)
- moved R20 1.12 mm to (238.9, 104.4)
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Routing:
- net /motor_driver/Fault2: track 28.4 -> 58.4 mm, vias 0 -> 2
- net /RX: track 36.2 -> 63.2 mm
- net Net-(U3-~{CHRG}): track 32.4 -> 13.7 mm, vias 0 -> 2
- net /IO0: track 58.0 -> 41.8 mm, vias 3 -> 2
- net /TX: track 44.0 -> 57.7 mm, vias 2 -> 4
- net /D-: track 5.99 -> 19.2 mm
- net Net-(U6-CPOUT): track 3.25 -> 16.2 mm
- net /motor_driver/Sl2: track 56.1 -> 44.0 mm
- net Net-(U6-AD0): track 4.28 -> 14.0 mm, vias 0 -> 2
- net /SRV_2: track 33.2 -> 24.5 mm
- net /EXI5: track 19.6 -> 27.2 mm, vias 0 -> 2
- net VBUS: track 50.7 -> 58.2 mm, vias 4 -> 2
- net GND: track 248.2 -> 255.2 mm, vias 17 -> 24
- net Net-(SW1A-C): track 30.9 -> 23.9 mm
- net Net-(U4-VDD): track 32.9 -> 26.3 mm, vias 2 -> 3
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
Commit message: 18-08-2025
Parts:
- added G***: LOGO, logo_3:logo_3, F.Cu at (258.9, 70.0)
- added G***: LOGO, logo_3:logo_3, F.Cu at (257.8, 133.8)
- added G***: LOGO, logo_3:logo_3, F.Cu at (194.1, 70.1)
- added G***: LOGO, logo_3:logo_3, F.Cu at (194.4, 133.9)
- added G***: LOGO, logo_20:logo_20, B.Cu at (227.8, 106.0)
Other:
- board text added: "+"
- board text added: "-"
