File: Modem_carrier_PCB/modem.kicad_sch (KiCad schematic)
At the start: 7 parts, among them J2 Conn_01x04_Socket, U3 SN74AVC4T245PW

Commit message: 27-12-2025_13:16
Parts:
- removed J2: Conn_01x04_Socket, symbol Connector:Conn_01x04_Socket
- added C11, C12, C13, C14: 100nF, symbol Device:C
- added D3: LED, symbol Device:LED
- added J2, J3: Conn_01x06_Socket, symbol Connector:Conn_01x06_Socket
- added J4: Conn_01x02_Socket, symbol Connector:Conn_01x02_Socket
- added J7: Conn_Coaxial, symbol Connector:Conn_Coaxial
- added Q1, Q2: 2N7002, PCM_Package_TO_SOT_SMD_AKL:SOT-23, symbol PCM_Transistor_MOSFET_AKL:2N7002
- added Q4: BC847, PCM_Package_TO_SOT_SMD_AKL:SOT-23, symbol PCM_Transistor_BJT_AKL:BC847
- added R10, R11: 100k, symbol Device:R
- added R17: 4.7k, symbol Device:R
- added R18, R8, R9: 47k, symbol Device:R
- added R19: 2.2k, symbol Device:R
- added U4: SN74AVC4T245PW, Package_SO:TSSOP-16_4.4x5mm_P0.65mm, symbol Logic_LevelTranslator:SN74AVC4T245PW
Connections:
- net GND: now also U3.14 (2~{OE}), U3.15 (1~{OE}), U3.2 (1DIR), U3.3 (2DIR), C11.2, C12.2, C13.2, C14.2, J2.6 (Pin_6), J3.6 (Pin_6), J7.2 (Ext), Q1.2 (S), Q2.2 (S), Q4.2 (E), R18.1, U4.14 (2~{OE}), U4.15 (1~{OE}), U4.2 (1DIR), U4.3 (2DIR), U4.8 (GND), U4.9 (GND)
- net VBAT: now also D3.2 (A)
- net VDD_EXT: now reaches U3.1 (VCCA)
- net VDD_EXT: now also U1.29 (VDD_EXT), C12.1, C13.1, R8.2, R9.1, U4.1 (VCCA)
- net at U3.10 (2B2): now also J2.5 (Pin_5)
- net at U3.11 (2B1): now also J2.4 (Pin_4)
- net at U3.12 (1B2): now also J2.3 (Pin_3)
- net at U3.13 (1B1): now also J2.2 (Pin_2)
- net at U3.16 (VCCB): now also C11.1, J2.1 (Pin_1)
- net at U3.4 (1A1): now also U1.36 (UART1_CTS)
- net at U3.5 (1A2): now also U1.37 (UART1_RTS)
- net at U3.6 (2A1): now also U1.35 (UART1_TXD)
- net at U3.7 (2A2): now also U1.34 (UART1_RXD)
- net PWRKEY_N: now reaches U1.15 (PWRKEY_N)
- net PWRKEY_N: now also Q2.3 (D), R8.1
- net RSTN: now reaches U1.17 (RSTN)
- net RSTN: now also Q1.3 (D), R9.2
- net STATUS: now reaches U1.20 (STATUS)
- net STATUS: now also R17.2
- net at U1.22 (UART2_RXD): now also U4.7 (2A2)
- net at U1.23 (UART2_TXD): now also U4.6 (2A1)
- net at U1.27 (UART0_TXD): now also U4.4 (1A1)
- net at U1.28 (UART0_RXD): now also U4.5 (1A2)
- net USIM_PRESENCE: now reaches U1.42 (USIM_PRESENCE)
- net USIM_VDD: now reaches U1.43 (USIM_VDD)
- net USIM_RST: now reaches U1.44 (USIM_RST)
- net USIM_DATA: now reaches U1.45 (USIM_DATA)
- net USIM_CLK: now reaches U1.46 (USIM_CLK)
- net at U1.60 (ANT_LTE): now also J7.1 (In)
- new net: Q2.1 (G), R11.1
- new net: J4.1 (Pin_1), R11.2
- new net: Q1.1 (G), R10.1
- new net: Q4.1 (B), R17.1, R18.2
- new net: Q4.3 (C), R19.2
- new net: C14.1, J3.1 (Pin_1), U4.16 (VCCB)
- new net: D3.1 (K), R19.1
- new net: J3.5 (Pin_5), U4.10 (2B2)
- new net: J3.4 (Pin_4), U4.11 (2B1)
- new net: J3.3 (Pin_3), U4.12 (1B2)
- new net: J3.2 (Pin_2), U4.13 (1B1)
- new net: J4.2 (Pin_2), R10.2
- no-connect marks 0 -> 35
Other:
- added sheet Sim card connections (untitled.kicad_sch)
- note added: "Use mosfet for safe switching from mcu"

Commit message: 27-12-2025_15:43
Parts:
- C10, C11, C12, C13, C14, C9: footprint (none) -> Capacitor_SMD:C_0603_1608Metric
- C7, C8: footprint (none) -> Capacitor_SMD:C_0805_2012Metric
- D3: footprint (none) -> LED_SMD:LED_0603_1608Metric
- J2, J3: footprint (none) -> Connector_PinHeader_1.27mm:PinHeader_1x06_P1.27mm_Vertical
- J4: footprint (none) -> Connector_PinHeader_1.27mm:PinHeader_1x02_P1.27mm_Vertical
- J7: footprint (none) -> U.FL-R-SMT_01_:HRS_U.FL-R-SMT_01_
- R10, R11, R18, R8, R9: footprint (none) -> Resistor_SMD:R_0805_2012Metric
- R17, R19: footprint (none) -> Resistor_SMD:R_0603_1608Metric
- U1: value ~ -> Cavli modem; footprint (none) -> Cavli_modem:C16QS
Changed lines of the file:
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@@
 			)
 		)
-		(column_widths 10.16)
-		(row_heights 2.54 2.54 2.54 2.54)
+		(column_widths 3.81)
+		(row_heights 2.54 2.54)
 		(cells
-			(table_cell "5"
-				(exclude_from_sim no)
-				(at 38.1 77.47 0)
-				(size 10.16 2.54)
-				(margins 0.9525 0.9525 0.9525 0.9525)
-				(span 1 1)
-				(fill
-					(type none)
-				)
-				(effects
-					(font
-						(size 1.27 1.27)
-					)
-					(justify left top)
-				)
-			)
-			(table_cell "4"
-				(exclude_from_sim no)
-				(at 38.1 80.01 0)
-				(size 10.16 2.54)
-				(margins 0.9525 0.9525 0.9525 0.9525)
-				(span 1 1)
-				(fill
-					(type none)
-				)
-				(effects
-					(font
-						(size 1.27 1.27)
-					)
-					(justify left top)
-				)
-			)
-			(table_cell "3"
+			(table_cell "2"
 				(exclude_from_sim no)
-				(at 38.1 82.55 0)
-				(size 10.16 2.54)
+				(at 17.78 31.75 0)
+				(size 3.81 2.54)
 				(margins 0.9525 0.9525 0.9525 0.9525)
 				(span 1 1)
@@
 				)
 			)
-			(table_cell "2"
+			(table_cell "1"
 				(exclude_from_sim no)
-				(at 38.1 85.09 0)
-				(size 10.16 2.54)
+				(at 17.78 34.29 0)
+				(size 3.81 2.54)
 				(margins 0.9525 0.9525 0.9525 0.9525)
 				(span 1 1)
@@
 			(table_cell "5"
 				(exclude_from_sim no)
-				(at 46.99 158.75 0)
+				(at 38.1 77.47 0)
 				(size 10.16 2.54)
 				(margins 0.9525 0.9525 0.9525 0.9525)
@@
 			(table_cell "4"
 				(exclude_from_sim no)
-				(at 46.99 161.29 0)
+				(at 38.1 80.01 0)
 				(size 10.16 2.54)
 				(margins 0.9525 0.9525 0.9525 0.9525)
@@
 			(table_cell "3"
 				(exclude_from_sim no)
-				(at 46.99 163.83 0)
+				(at 38.1 82.55 0)
 				(size 10.16 2.54)
 				(margins 0.9525 0.9525 0.9525 0.9525)
@@
 			(table_cell "2"
 				(exclude_from_sim no)
-				(at 46.99 166.37 0)
+				(at 38.1 85.09 0)
 				(size 10.16 2.54)
 				(margins 0.9525 0.9525 0.9525 0.9525)
@@
 			)
 		)
-		(column_widths 3.81)
-		(row_heights 2.54 2.54)
+		(column_widths 10.16)
+		(row_heights 2.54 2.54 2.54 2.54)
 		(cells
-			(table_cell "2"
+			(table_cell "5"
 				(exclude_from_sim no)
-				(at 17.78 31.75 0)
-				(size 3.81 2.54)
+				(at 46.99 158.75 0)
+				(size 10.16 2.54)
 				(margins 0.9525 0.9525 0.9525 0.9525)
 				(span 1 1)
@@
 				)
 			)
-			(table_cell "1"
+			(table_cell "4"
 				(exclude_from_sim no)
-				(at 17.78 34.29 0)
-				(size 3.81 2.54)
+				(at 46.99 161.29 0)
+				(size 10.16 2.54)
+				(margins 0.9525 0.9525 0.9525 0.9525)
+				(span 1 1)
+				(fill
+					(type none)
+				)
+				(effects
+					(font
+						(size 1.27 1.27)
+					)
+					(justify left top)
+				)
+			)
+			(table_cell "3"
+				(exclude_from_sim no)
+				(at 46.99 163.83 0)
+				(size 10.16 2.54)
+				(margins 0.9525 0.9525 0.9525 0.9525)
+				(span 1 1)
+				(fill
+					(type none)
+				)
+				(effects
+					(font
+						(size 1.27 1.27)
+					)
+					(justify left top)
+				)
+			)
+			(table_cell "2"
+				(exclude_from_sim no)
+				(at 46.99 166.37 0)
+				(size 10.16 2.54)
 				(margins 0.9525 0.9525 0.9525 0.9525)
 				(span 1 1)
@@
 			)
 		)
-		(property "Footprint" ""
+		(property "Footprint" "Resistor_SMD:R_0805_2012Metric"
 			(at 53.34 41.402 90)
 			(effects
@@
 			)
 		)
-		(property "Footprint" ""
+		(property "Footprint" "Capacitor_SMD:C_0603_1608Metric"
 			(at 47.9552 143.51 0)
 			(effects
@@
 			)
 		)
-		(property "Footprint" ""
+		(property "Footprint" "Capacitor_SMD:C_0603_1608Metric"
 			(at 56.8452 143.51 0)
 			(effects
@@
 			)
 		)
-		(property "Footprint" ""
+		(property "Footprint" "Capacitor_SMD:C_0805_2012Metric"
 			(at 40.3352 143.51 0)
 			(effects
@@
 			)
 		)
-		(property "Footprint" ""
+		(property "Footprint" "Capacitor_SMD:C_0603_1608Metric"
 			(at 84.7852 115.57 0)
 			(effects
@@
 			)
 		)
-		(property "Footprint" ""
+		(property "Footprint" "Capacitor_SMD:C_0603_1608Metric"
 			(at 79.7052 170.18 0)
 			(effects
@@
 			)
 		)
-		(property "Footprint" ""
+		(property "Footprint" "Resistor_SMD:R_0603_1608Metric"
 			(at 242.062 35.56 90)
 			(effects
@@
 			)
 		)
-		(property "Footprint" ""
+		(property "Footprint" "U.FL-R-SMT_01_:HRS_U.FL-R-SMT_01_"
 			(at 171.45 57.15 0)
 			(effects
@@
 			)
 		)
-		(property "Footprint" ""
+		(property "Footprint" "Resistor_SMD:R_0805_2012Metric"
 			(at 237.49 56.642 90)
 			(effects
@@
 			)
 		)
-		(property "Footprint" ""
+		(property "Footprint" "Resistor_SMD:R_0805_2012Metric"
 			(at 81.28 18.542 90)
 			(effects
@@
 			)
 		)
-		(property "Footprint" ""
+		(property "Footprint" "Resistor_SMD:R_0805_2012Metric"
 			(at 46.99 26.162 90)
 			(effects
@@
 			)
 		)
-		(property "Footprint" ""
+		(property "Footprint" "Resistor_SMD:R_0805_2012Metric"
 			(at 85.09 38.608 90)
 			(effects
@@
 			)
 		)
-		(property "Footprint" ""
+		(property "Footprint" "Connector_PinHeader_1.27mm:PinHeader_1x06_P1.27mm_Vertical"
 			(at 71.12 142.24 0)
 			(effects
@@
 			)
 		)
-		(property "Footprint" ""
+		(property "Footprint" "Capacitor_SMD:C_0603_1608Metric"
 			(at 99.06 162.8648 0)
 			(effects
@@
 			)
 		)
-		(property "Footprint" ""
+		(property "Footprint" "Capacitor_SMD:C_0603_1608Metric"
 			(at 99.06 105.7148 0)
 			(effects
@@
 			)
 		)
-		(property "Footprint" ""
+		(property "Footprint" "Connector_PinHeader_1.27mm:PinHeader_1x02_P1.27mm_Vertical"
 			(at 38.1 30.48 0)
 			(effects
@@
 			)
 		)
-		(property "Value" "~"
+		(property "Value" "Cavli modem"
 			(at 132.715 36.83 0)
 			(effects
@@
 			)
 		)
-		(property "Footprint" ""
+		(property "Footprint" "Cavli_modem:C16QS"
 			(at 121.92 50.8 0)
 			(effects
@@
 			)
 		)
-		(property "Footprint" ""
+		(property "Footprint" "LED_SMD:LED_0603_1608Metric"
 			(at 243.84 25.4 0)
 			(effects
@@
 			)
 		)
-		(property "Footprint" ""
+		(property "Footprint" "Connector_PinHeader_1.27mm:PinHeader_1x06_P1.27mm_Vertical"
 			(at 68.58 83.82 0)
 			(effects
@@
 			)
 		)
-		(property "Footprint" ""
+		(property "Footprint" "Capacitor_SMD:C_0805_2012Metric"
 			(at 32.7152 143.51 0)
 			(effects
@@
 			)
 		)
-		(property "Footprint" ""
+		(property "Footprint" "Resistor_SMD:R_0603_1608Metric"
 			(at 227.33 46.482 90)
 			(effects
