File: Modem_carrier_PCB/Modem_carrier_PCB.kicad_pcb (KiCad board)
At the start: 2 copper layers, 56 parts, among them J1 USB_C_Receptacle_PowerOnly_6P, J2 Conn_01x06_Socket, J3 Conn_01x06_Socket, J4 Conn_01x02_Socket, J5 JAE_SIM_Card_SF72S006, J6 Conn_01x01_Socket, J7 Conn_Coaxial, Q1 2N7002, Q2 2N7002, Q3 2N7002, Q4 BC847, U1 Cavli modem, U2 AP62250Z6, U3 SN74AVC4T245PW, U4 SN74AVC4T245PW

Commit message: 27-12-2025_17:50
Parts:
- moved D2 123.8 mm to (216.8, 80.8)
- moved J5 122.2 mm to (222.9, 88.7)
- moved J6 113.7 mm to (213.2, 96.8)
- moved R12 106.6 mm to (214.8, 85.2), turned to -90 degrees
- moved C7 106.0 mm to (205.4, 96.5), turned to 180 degrees
- moved C8 105.9 mm to (205.4, 98.7), turned to 180 degrees
- moved Q3 104.4 mm to (212.6, 92.2)
- moved R13 104.3 mm to (211.8, 78.1), turned to 180 degrees
- moved R15 104.2 mm to (211.8, 84.2), turned to 180 degrees
- moved R14 104.1 mm to (211.8, 82.3)
- moved R16 104.1 mm to (211.8, 87.7), turned to 180 degrees
- moved C16 103.6 mm to (214.8, 78.1), turned to 180 degrees
- moved C17 103.3 mm to (215.1, 87.8), turned to 90 degrees
- moved C18 99.9 mm to (211.5, 85.9)
- moved C15 99.9 mm to (211.5, 80.4), turned to 180 degrees
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Routing:
- net GND: track 0.00 -> 341.8 mm, vias 0 -> 14
- net /Modem/VDD_EXT: track 0.00 -> 70.0 mm, vias 0 -> 3
- net VBAT: track 0.00 -> 58.9 mm
- net Net-(U1-UART1_CTS): track 0.00 -> 38.6 mm, vias 0 -> 2
- net Net-(D2-L4): track 0.00 -> 35.1 mm, vias 0 -> 2
- net /Modem/USIM_PRESENCE: track 0.00 -> 35.1 mm
- net Net-(U1-UART1_TXD): track 0.00 -> 33.9 mm, vias 0 -> 2
- net Net-(U1-UART1_RTS): track 0.00 -> 32.5 mm, vias 0 -> 2
- net /Modem/USIM_VDD: track 0.00 -> 29.4 mm
- net Net-(U1-UART1_RXD): track 0.00 -> 28.8 mm, vias 0 -> 2
- net Net-(U1-UART0_TXD): track 0.00 -> 26.9 mm, vias 0 -> 2
- net /Modem/PWRKEY_N: track 0.00 -> 26.1 mm, vias 0 -> 2
- net Net-(D2-L3): track 0.00 -> 24.3 mm, vias 0 -> 2
- net +5V: track 0.00 -> 22.7 mm
- net Net-(U1-UART0_RXD): track 0.00 -> 22.6 mm, vias 0 -> 2
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- added copper zone on B.Cu, net GND
Other:
- board outline added: 57.5 x 62.4 mm
- board text added: "C16QS-HARSHIL_SUTHAR-v1"
