File: ESP32_based_dev_board/ESP32_based_dev_board.kicad_pcb (KiCad board)
At the start: 4 copper layers, 83.7 x 54.8 mm, 92 parts, among them J1 SS-52400-002, J2 B2B-PH-SM4-TB, J3 GSD090012SEU, J4 Conn_01x04_Pin, J5 Conn_01x05_Pin, Q1 TEMT6000X01, Q2 BC817, Q3 BC817, U1 MCP73871-2CAI_ML, U2 BME280, U3 ESP32-C3-WROOM-02-H4, U4 CP2102N-Axx-xQFN20, U5 USBLC6-2SC6, U6 W25Q32JVSSIQ, U7 MAX4466EXK

Commit message: 05-01-2026_20:41
Parts:
- added C23: 0.1u, Capacitor_SMD:C_0805_2012Metric, F.Cu at (185.8, 93.2)
- added C24: 10n, Capacitor_SMD:C_0805_2012Metric, F.Cu at (181.0, 89.8)
- added C25: 10n, Capacitor_SMD:C_0805_2012Metric, F.Cu at (232.5, 81.8)
- added FB1: Ferrite_Bead, ESP32_Proj_Footprints:BEADC2012X105N, F.Cu at (171.8, 123.2)
- added R17: 35WR100KLFTR, ESP32_Proj_Footprints:TRIM_35WR100KLFTR, F.Cu at (175.0, 91.5)
- C19: value 1u -> 10u
- C20: value 0.1u -> 100pF
- R30: value 10K -> 1K
- R31: value 100K -> 22K
- moved Q1 3.29 mm to (181.2, 93.2)
- moved R23 1.41 mm to (183.5, 89.8), turned to 90 degrees
Connections:
- Q1 pad 1: GND -> /ESP32-C3-02/PHOTO_C
- Q1 pad 3: /ESP32-C3-02/PHOTO_C -> +3.3V
- R23 pad 1: +3.3V -> /ESP32-C3-02/PHOTO_C
- R23 pad 2: /ESP32-C3-02/PHOTO_C -> GND
- R31 pad 2: /ESP32-C3-02/MIC_OUT -> Net-(R17-Pad3)
- U1 pad 1: +5V -> Net-(FB1-Pad1)
- U1 pad 20: +5V -> Net-(FB1-Pad1)
- U3 pad 18: /ESP32-C3-02/CS_SD -> /ESP32-C3-02/MIC_OUT
- U3 pad 4: /ESP32-C3-02/MIC_OUT -> /ESP32-C3-02/CS_SD
Routing:
- net /ESP32-C3-02/MIC_OUT: track 38.4 -> 78.4 mm
- net Net-(R17-Pad3): track 0.00 -> 21.8 mm
- net /ESP32-C3-02/CS_SD: track 27.0 -> 38.4 mm
- net /ESP32-C3-02/PHOTO_C: track 52.3 -> 58.4 mm
- net GND: track 156.7 -> 161.1 mm, vias 41 -> 43
- net Net-(FB1-Pad1): track 0.00 -> 3.27 mm
- net +3.3V: track 72.2 -> 74.5 mm
- net +5V: track 29.0 -> 26.9 mm
- added copper zone on F.Cu, net Net-(FB1-Pad1)
- removed copper zone on F.Cu, net +5V
Other:
- board size 83.7 x 54.8 mm -> 84.5 x 54.8 mm
- board text added: "USB"
