File: ESP32_based_dev_board/ESP32_based_dev_board.kicad_sch (KiCad schematic)
At the start: 0 parts

Commit message: 05-01-2026_19:28
Parts:
- added C1, C2, C5: 0.1u, Capacitor_SMD:C_0805_2012Metric, symbol Device:C
- added C3, C4: 10u, ESP32_Proj_Footprints:T491A, symbol Device:C_Polarized
- added C6: 1u, Capacitor_SMD:C_0805_2012Metric, symbol Device:C
- added F1: 0ZCH0110AF2E, ESP32_Proj_Footprints:FUSC3226X100N, symbol 0ZCH0110AF2E:0ZCH0110AF2E
- added J1: SS-52400-002, ESP32_Proj_Footprints:BELFUSE_SS-52400-002, symbol SS-52400-002:SS-52400-002
- added J2: B2B-PH-SM4-TB, B2B-PH-SM4-TB:JST_B2B-PH-SM4-TB, symbol B2B-PH-SM4-TB:B2B-PH-SM4-TB
- added LED1, LED4: LTST-C170KRKT, ESP32_Proj_Footprints:LEDC2012X120N, symbol LTST-C170KRKT:LTST-C170KRKT
- added LED2: LTST-C170GKT, ESP32_Proj_Footprints:LEDC2012X120N, symbol LTST-C170GKT:LTST-C170GKT
- added LED3: LTST-C170TBKT, ESP32_Proj_Footprints:LEDC2012X120N, symbol LTST-C170TBKT:LTST-C170TBKT
- added R1, R2: 10K, Resistor_SMD:R_0805_2012Metric, symbol Device:R
- added R10, R7, R8, R9: 470, Resistor_SMD:R_0805_2012Metric, symbol Device:R
- added R3, R4: 5K1, Resistor_SMD:R_0805_2012Metric, symbol Device:R
- added R5: 2K, Resistor_SMD:R_0805_2012Metric, symbol Device:R
- added R6: 20K, Resistor_SMD:R_0805_2012Metric, symbol Device:R
- added U1: MCP73871-2CAI_ML, ESP32_Proj_Footprints:QFN50P400X400X100-21N, symbol MCP73871-2CAI_ML:MCP73871-2CAI_ML
- added VR1: LM1117MPX-3.3, ESP32_Proj_Footprints:VREG_LM1117MPX-3.3, symbol LM1117MPX-3.3:LM1117MPX-3.3
Connections:
- new net: LED3.1 (K), R7.1
- new net: LED2.1 (K), R8.2
- new net: R6.1, U1.12 (PROG3)
- new net: R5.1, U1.13 (PROG1)
- new net: R2.2, U1.5 (THERM)
- new net: R1.1, U1.9 (~{TE})
- new net: LED1.1 (K), R9.1
- new net: J1.A5 (CC1), R4.2
- new net: J1.B5 (CC2), R3.2
- new net: LED4.1 (K), R10.1
- new net +3.3V: C4.1, C5.1, LED4.2 (A), VR1.2 (VOUT_2), VR1.4 (VOUT_4)
- new net +5V: C2.1, C3.1, U1.1 (OUT), U1.20 (OUT), VR1.3 (VIN)
- new net +5V_USB: C6.2, F1.2, LED1.2 (A), LED2.2 (A), LED3.2 (A), U1.17 (CE), U1.18 (IN), U1.19 (IN), U1.2 (VPCC), U1.4 (PROG2)
- new net CHARGED: R8.1, U1.8 (STAT1/~{LBO})
- new net CHARGING: R9.2, U1.6 (~{PG})
- new net CHARGING_POWER_GOOD: R7.2, U1.7 (STAT2)
- new net GND: C1.2, C2.2, C3.2, C4.2, C5.2, C6.1, J1.A1 (GNDA1), J1.A12 (GNDA2), J1.B1 (GNDB1), J1.B12 (GNDB2), J1.G1 (GND/SHIELD), J1.G2 (GND/SHIELD), J1.G3 (GND/SHIELD), J1.G4 (GND/SHIELD), J1.S1 (GND/SHIELD), J1.S2 (GND/SHIELD), J1.S3 (GND/SHIELD), J1.S4 (GND/SHIELD), J2.1, R1.2, R10.2, R2.1, R3.1, R4.1, R5.2, R6.2, U1.10 (VSS), U1.11 (VSS), U1.21 (VSS), U1.3 (SEL), VR1.1 (GND)
- new net USB_DN: J1.A7 (DN1), J1.B7 (DN2)
- new net USB_DP: J1.A6 (DP1), J1.B6 (DP2)
- new net VBAT: J2.2, U1.14 (VBAT), U1.15 (VBAT), U1.16 (VBAT_SENSE)
- new net VBUS: C1.1, F1.1, J1.A4 (VBUSA1), J1.A9 (VBUSA2), J1.B4 (VBUSB1), J1.B9 (VBUSB2)
- no-connect marks 0 -> 10
Other:
- added sheet ESP32-C3-02 (esp32-c3-02.kicad_sch)
- note added: "Battery JST connector"
- note added: "Lipo battery charger"
- note added: "Low drop out (LDO) voltage regulator"
- note added: "Power indicator LED"
- note added: "USB-C connector"
- title: (none) -> ESP32 sensor board

Commit message: 05-01-2026_20:41
Parts:
- added FB1: Ferrite_Bead, ESP32_Proj_Footprints:BEADC2012X105N, symbol PCM_Device_AKL:Ferrite_Bead
Connections:
- net +5V: now also FB1.2; no longer U1.1 (OUT), U1.20 (OUT)
- new net: FB1.1, U1.1 (OUT), U1.20 (OUT)
Changed lines of the file:
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@@
 	(wire
 		(pts
-			(xy 250.19 26.67) (xy 248.92 26.67)
+			(xy 248.92 26.67) (xy 252.73 26.67)
 		)
 		(stroke
@@
 	(wire
 		(pts
-			(xy 250.19 22.86) (xy 250.19 26.67)
-		)
-		(stroke
-			(width 0)
-			(type default)
-		)
-	)
-	(wire
-		(pts
 			(xy 99.06 93.98) (xy 105.41 93.98)
 		)
@@
 	(wire
 		(pts
+			(xy 266.7 26.67) (xy 266.7 24.13)
+		)
+		(stroke
+			(width 0)
+			(type default)
+		)
+	)
+	(wire
+		(pts
 			(xy 218.44 124.46) (xy 218.44 121.92)
 		)
@@
 	(wire
 		(pts
+			(xy 260.35 26.67) (xy 266.7 26.67)
+		)
+		(stroke
+			(width 0)
+			(type default)
+		)
+	)
+	(wire
+		(pts
 			(xy 167.64 116.84) (xy 167.64 121.92)
 		)
@@
 	(symbol
 		(lib_id "power:+5V")
-		(at 250.19 22.86 0)
+		(at 266.7 24.13 0)
 		(unit 1)
 		(exclude_from_sim no)
@@
 		(fields_autoplaced yes)
 		(property "Reference" "#PWR020"
-			(at 250.19 26.67 0)
+			(at 266.7 27.94 0)
 			(effects
 				(font
@@
 		)
 		(property "Value" "+5V"
-			(at 250.19 17.78 0)
+			(at 266.7 19.05 0)
 			(effects
 				(font
@@
 		)
 		(property "Footprint" ""
-			(at 250.19 22.86 0)
+			(at 266.7 24.13 0)
 			(effects
 				(font
@@
 		)
 		(property "Datasheet" ""
-			(at 250.19 22.86 0)
+			(at 266.7 24.13 0)
 			(effects
 				(font
@@
 		)
 		(property "Description" "Power symbol creates a global label with name \"+5V\""
-			(at 250.19 22.86 0)
+			(at 266.7 24.13 0)
 			(effects
 				(font
@@
 					(unit 1)
 				)
+			)
+		)
+	)
+	(symbol
+		(lib_id "PCM_Device_AKL:Ferrite_Bead")
+		(at 256.54 26.67 0)
+		(unit 1)
+		(exclude_from_sim no)
+		(in_bom yes)
+		(on_board yes)
+		(dnp no)
+		(property "Reference" "FB1"
+			(at 256.54 21.336 0)
+			(effects
+				(font
+					(size 1.27 1.27)
+				)
+			)
+		)
+		(property "Value" "Ferrite_Bead"
+			(at 256.54 23.876 0)
+			(effects
+				(font
+					(size 1.27 1.27)
+				)
+			)
+		)
+		(property "Footprint" "ESP32_Proj_Footprints:BEADC2012X105N"
+			(at 256.54 23.368 0)
+			(effects
+				(font
+					(size 1.27 1.27)
+				)
+				(hide yes)
+			)
+		)
+		(property "Datasheet" "~"
+			(at 256.54 26.67 90)
+			(effects
+				(font
+					(size 1.27 1.27)
+				)
+				(hide yes)
+			)
+		)
+		(property "Description" "Ferrite bead, Alternate KiCAD Library"
+			(at 256.54 26.67 0)
+			(effects
+				(font
+					(size 1.27 1.27)
+				)
+				(hide yes)
+			)
+		)
+		(pin "2"
+		)
+		(pin "1"
+		)
+		(instances
+			(project ""
+				(path "/5293f698-2317-4ac2-8b7a-334d10b8a673"
+					(reference "FB1")
+					(unit 1)
+				)
