File: ESP32_based_dev_board/esp32-c3-02.kicad_sch (KiCad schematic)
At the start: 30 parts, among them J3 GSD090012SEU, U3 ESP32-C3-WROOM-02-H4, U4 CP2102N-Axx-xQFN20, U5 USBLC6-2SC6, U6 W25Q32JVSSIQ

Commit message: 05-01-2026_20:41
Connections:
- net CS_SD: now also U3.4 (IO5); no longer U3.18 (IO0)
- net MIC_OUT: now also U3.18 (IO0); no longer U3.4 (IO5)
Changed lines of the file:
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@@
 	)
 	(label "CS_SD"
-		(at 194.31 44.45 180)
+		(at 194.31 57.15 180)
 		(effects
 			(font
@@
 	)
 	(label "MIC_OUT"
-		(at 194.31 57.15 180)
+		(at 194.31 44.45 180)
 		(effects
 			(font
