File: ESP32_based_dev_board/sensors.kicad_sch (KiCad schematic)
At the start: 19 parts, among them Q1 TEMT6000X01, U2 BME280, U7 MAX4466EXK

Commit message: 05-01-2026_20:41
Parts:
- added C23: 0.1u, Capacitor_SMD:C_0805_2012Metric, symbol Device:C
- added C24, C25: 10n, Capacitor_SMD:C_0805_2012Metric, symbol Device:C
- added R17: 35WR100KLFTR, ESP32_Proj_Footprints:TRIM_35WR100KLFTR, symbol 35WR100KLFTR:35WR100KLFTR
- C19: value 1u -> 10u
- C20: value 0.1u -> 100pF
- R30: value 10K -> 1K
- R31: value 100K -> 22K
Connections:
- net +3.3V: now also Q1.3, C23.1; no longer R23.1
- net GND: now also R23.2, C23.2, C24.2, C25.2; no longer Q1.1
- net MIC_OUT: now also R17.1, R17.2; no longer R31.2
- net PHOTO_C: now also Q1.1, R23.1, C24.1, C25.1; no longer Q1.3, R23.2
- new net: R17.3, R31.2
Other:
- moved on the sheet: C20, Q1, R23, R31
